File: Arduino Shield/Bomb.kicad_sch (KiCad schematic)
At the start: 6 parts, among them J1 Digital/PWM, J2 I2C Out, J3 Power, J4 Logic, U1 ATtiny85

Commit message: Added LED shield hardware files
Parts:
- C1: footprint (none) -> Capacitor_SMD:C_0504_1310Metric_Pad0.83x1.28mm_HandSolder
Changed lines of the file:
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@@
   (symbol (lib_name "GND_4") (lib_id "power:GND") (at 134.62 97.79 0) (unit 1)
     (in_bom yes) (on_board yes) (fields_autoplaced)
-    (property "Reference" "#PWR?" (id 0) (at 134.62 104.14 0)
+    (property "Reference" "#PWR0108" (id 0) (at 134.62 104.14 0)
       (effects (font (size 1.27 1.27)) hide)
     )
@@
   (symbol (lib_id "power:+5V") (at 134.62 85.09 0) (unit 1)
     (in_bom yes) (on_board yes) (fields_autoplaced)
-    (property "Reference" "#PWR?" (id 0) (at 134.62 88.9 0)
+    (property "Reference" "#PWR0109" (id 0) (at 134.62 88.9 0)
       (effects (font (size 1.27 1.27)) hide)
     )
@@
     )
     (property "Value" "C" (id 1) (at 138.43 92.7099 0)
-      (effects (font (size 1.27 1.27)) (justify left))
-    )
-    (property "Footprint" "" (id 2) (at 135.5852 95.25 0)
+      (effects (font (size 1.27 1.27)) (justify left) hide)
+    )
+    (property "Footprint" "Capacitor_SMD:C_0504_1310Metric_Pad0.83x1.28mm_HandSolder" (id 2) (at 135.5852 95.25 0)
       (effects (font (size 1.27 1.27)) hide)
     )
@@
   (symbol (lib_name "GND_3") (lib_id "power:GND") (at 87.63 91.44 0) (unit 1)
     (in_bom yes) (on_board yes) (fields_autoplaced)
-    (property "Reference" "#PWR?" (id 0) (at 87.63 97.79 0)
+    (property "Reference" "#PWR0107" (id 0) (at 87.63 97.79 0)
       (effects (font (size 1.27 1.27)) hide)
     )
@@
       (reference "#PWR0106") (unit 1) (value "GND") (footprint "")
     )
+    (path "/be7b6f0b-089e-451d-ad44-f2f61bc1d67e"
+      (reference "#PWR0107") (unit 1) (value "GND") (footprint "")
+    )
     (path "/33d7bb50-7f98-4f0d-aab9-331f7ac648c8"
-      (reference "#PWR?") (unit 1) (value "GND") (footprint "")
+      (reference "#PWR0108") (unit 1) (value "GND") (footprint "")
     )
     (path "/64fd6d22-94c2-46a8-af3d-36696e98cb48"
-      (reference "#PWR?") (unit 1) (value "+5V") (footprint "")
-    )
-    (path "/be7b6f0b-089e-451d-ad44-f2f61bc1d67e"
-      (reference "#PWR?") (unit 1) (value "GND") (footprint "")
+      (reference "#PWR0109") (unit 1) (value "+5V") (footprint "")
     )
     (path "/9ce64185-fda7-4aae-b239-f4139326ce56"
-      (reference "C1") (unit 1) (value "C") (footprint "")
+      (reference "C1") (unit 1) (value "C") (footprint "Capacitor_SMD:C_0504_1310Metric_Pad0.83x1.28mm_HandSolder")
     )
     (path "/00000000-0000-0000-0000-000056d72368"

Commit message: Widened the pads of C1 in the arduino shield, switched the pinout of the i2c out, adjusted the size of the arduino shield board
Connections:
- net SCL/A5: now also J2.4 (Pin_4); no longer J2.3 (Pin_3)
- net SDA/A4: now also J2.3 (Pin_3); no longer J2.4 (Pin_4)
Changed lines of the file:
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@@
-    (effects (font (size 1.27 1.27)) (justify left bottom))
-  )
-  (label "SDA{slash}A4" (at 21.59 97.79 0)
-    (effects (font (size 1.27 1.27)) (justify left bottom))
-  )
-  (label "SCL{slash}A5" (at 21.59 95.25 0)
     (effects (font (size 1.27 1.27)) (justify left bottom))
   )
@@
     (effects (font (size 1.27 1.27)) (justify right bottom))
   )
+  (label "SCL{slash}A5" (at 21.59 97.79 0)
+    (effects (font (size 1.27 1.27)) (justify left bottom))
+  )
   (label "12" (at 81.28 96.52 180)
     (effects (font (size 1.27 1.27)) (justify right bottom))
@@
     (effects (font (size 1.27 1.27)) (justify right bottom))
   )
+  (label "SDA{slash}A4" (at 21.59 95.25 0)
+    (effects (font (size 1.27 1.27)) (justify left bottom))
+  )
   (label "*11" (at 140.97 31.75 180)
